File: sensors.kicad_sch (KiCad schematic)
At the start: 6 parts, among them U6 ICM-42688-P, U7 ICP-10111

Commit message: add lots of test points
Parts:
- added TP10: TestPoint, symbol Connector:TestPoint
Connections:
- net MOTION_INT: now also TP10.1
Changed lines of the file:
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@@
+	)
+	(junction
+		(at 35.56 44.45)
+		(diameter 0)
+		(color 0 0 0 0)
 	)
 	(junction
@@
 	(wire
 		(pts
+			(xy 35.56 44.45) (xy 48.26 44.45)
+		)
+		(stroke
+			(width 0)
+			(type default)
+		)
+	)
+	(wire
+		(pts
 			(xy 44.45 49.53) (xy 44.45 52.07)
 		)
@@
 	(wire
 		(pts
-			(xy 40.64 44.45) (xy 48.26 44.45)
+			(xy 31.75 44.45) (xy 35.56 44.45)
 		)
 		(stroke
@@
 	(hierarchical_label "MOTION_INT"
 		(shape output)
-		(at 40.64 44.45 180)
+		(at 31.75 44.45 180)
 		(fields_autoplaced yes)
 		(effects
@@
 					(unit 1)
 				)
+			)
+		)
+	)
+	(symbol
+		(lib_id "Connector:TestPoint")
+		(at 35.56 44.45 0)
+		(unit 1)
+		(exclude_from_sim no)
+		(in_bom yes)
+		(on_board yes)
+		(dnp no)
+		(fields_autoplaced yes)
+		(property "Reference" "TP10"
+			(at 38.1 39.8779 0)
+			(effects
+				(font
+					(size 1.27 1.27)
+				)
+				(justify left)
+			)
+		)
+		(property "Value" "TestPoint"
+			(at 38.1 42.4179 0)
+			(effects
+				(font
+					(size 1.27 1.27)
+				)
+				(justify left)
+			)
+		)
+		(property "Footprint" ""
+			(at 40.64 44.45 0)
+			(effects
+				(font
+					(size 1.27 1.27)
+				)
+				(hide yes)
+			)
+		)
+		(property "Datasheet" "~"
+			(at 40.64 44.45 0)
+			(effects
+				(font
+					(size 1.27 1.27)
+				)
+				(hide yes)
+			)
+		)
+		(property "Description" "test point"
+			(at 35.56 44.45 0)
+			(effects
+				(font
+					(size 1.27 1.27)
+				)
+				(hide yes)
+			)
+		)
+		(pin "1"
+		)
+		(instances
+			(project "OpenBikeComputer"
+				(path "/110ea5a2-03d6-426d-b79f-fcb4ea6cee9d/7aa00029-f5f2-4535-b444-7e5f9da482b1"
+					(reference "TP10")
+					(unit 1)
+				)
