File: OpenBikeComputer.kicad_pcb (KiCad board)
At the start: 4 copper layers, 45 x 60 mm, 49 parts, among them J1 USB_C_Receptacle_USB2.0_14P, J3 Conn_01x30_Socket, J4 Micro_SD_Card_Det1, J6 Conn_01x03_Pin, J7 RFShield_TwoPieces, J8 Conn_01x02_Socket, SW1 SW_Push, SW2 SW_Push, SW3 SW_Push, SW4 SW_Push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

Commit message: add sd card model and stuff
Parts:
- moved U6 33.8 mm to (153.0, 132.5)
- moved U7 33.8 mm to (158.9, 132.4)
- moved J8 0.95 mm to (157.8, 80.0)
Changed lines of the file:
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@@
 			)
 		)
+		(model "${KIPRJMOD}/Library.pretty/packages3d/tf-card.step"
+			(offset
+				(xyz 0 -2.6 0)
+			)
+			(scale
+				(xyz 1 1 1)
+			)
+			(rotate
+				(xyz 0 0 -90)
+			)
+		)
 	)
 	(footprint "Capacitor_SMD:C_0201_0603Metric"
@@
 	(footprint "Library:LGA-14_L3.0-W2.5-P0.50-TL"
 		(layer "F.Cu")
-		(at 186.75 133)
+		(at 152.987998 132.499936)
 		(descr "LGA-14_L3.0-W2.5-P0.50-TL footprint")
 		(tags "LGA-14_L3.0-W2.5-P0.50-TL footprint C1850418")
@@
 	(footprint "Library:PSON65P250X200X100-8N"
 		(layer "F.Cu")
-		(at 192.625 132.87)
+		(at 158.862998 132.369936)
 		(property "Reference" "U7"
 			(at 0.02672 -1.906224 0)
@@
 	(footprint "Connector_JST:JST_PH_S2B-PH-K_1x02_P2.00mm_Horizontal"
 		(layer "B.Cu")
-		(at 156.9 80 90)
+		(at 157.85 80 90)
 		(descr "JST PH series connector, S2B-PH-K (http://www.jst-mfg.com/product/pdf/eng/ePH.pdf), generated with kicad-footprint-generator")
 		(tags "connector JST PH top entry")
