File: display.kicad_sch (KiCad schematic)
At the start: 12 parts, among them J3 Conn_01x30_Socket, U5 FAN5331SX

Commit message: route PMIC
Connections:
- net 3.0V renamed +3V0
Other:
- note added: "This schematic was made for a NHD-1.91-176176B OLED display. It needs 17V on its display supply power supply. If you're using a different display, CHECK THE DATASHEET."
- note removed: "This schematic was made for a REX128128AWAP3N00000 128x128 monochrome OLED display. It needs 14.5V on its display supply power supply. If you're using a different display, CHECK THE DATASHEET."
- note removed: "We're using SPI so both pins are connected to VSS"
Changed lines of the file:
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@@
 		)
 	)
-	(text "This schematic was made for a REX128128AWAP3N00000 128x128 monochrome OLED display.\n\nIt needs 14.5V on its display supply power supply.\n\nIf you're using a different display, CHECK THE DATASHEET."
+	(text "This schematic was made for a NHD-1.91-176176B OLED display.\n\nIt needs 17V on its display supply power supply.\n\nIf you're using a different display, CHECK THE DATASHEET."
 		(exclude_from_sim no)
 		(at 201.168 70.866 0)
@@
 		)
 	)
-	(text "We're using SPI\nso both pins are connected to VSS"
-		(exclude_from_sim no)
-		(at 178.562 84.074 0)
+	(global_label "VOUT"
+		(shape input)
+		(at 154.94 125.73 180)
+		(fields_autoplaced yes)
 		(effects
 			(font
 				(size 1.27 1.27)
 			)
+			(justify right)
+		)
+		(property "Intersheetrefs" "${INTERSHEET_REFS}"
+			(at 147.2376 125.73 0)
+			(effects
+				(font
+					(size 1.27 1.27)
+				)
+				(justify right)
+				(hide yes)
+			)
 		)
 	)
 	(global_label "VOUT"
-		(shape input)
-		(at 154.94 125.73 180)
+		(shape output)
+		(at 24.13 73.66 180)
 		(fields_autoplaced yes)
 		(effects
@@
 		)
 		(property "Intersheetrefs" "${INTERSHEET_REFS}"
-			(at 147.2376 125.73 0)
+			(at 16.4276 73.66 0)
 			(effects
 				(font
@@
 		)
 	)
-	(global_label "VOUT"
-		(shape output)
-		(at 24.13 73.66 180)
+	(hierarchical_label "DISPLAY_SHDN"
+		(shape input)
+		(at 93.98 105.41 270)
 		(fields_autoplaced yes)
 		(effects
@@
 			(justify right)
 		)
-		(property "Intersheetrefs" "${INTERSHEET_REFS}"
-			(at 16.4276 73.66 0)
-			(effects
-				(font
-					(size 1.27 1.27)
-				)
-				(justify right)
-				(hide yes)
-			)
-		)
-	)
-	(hierarchical_label "DISPLAY_SHDN"
+	)
+	(hierarchical_label "MOSI"
 		(shape input)
-		(at 93.98 105.41 270)
+		(at 147.32 107.95 180)
 		(fields_autoplaced yes)
 		(effects
@@
 		)
 	)
-	(hierarchical_label "1.8V"
-		(shape passive)
-		(at 152.4 77.47 180)
+	(hierarchical_label "SCLK"
+		(shape input)
+		(at 147.32 105.41 180)
 		(fields_autoplaced yes)
 		(effects
@@
 		)
 	)
-	(hierarchical_label "MOSI"
-		(shape input)
-		(at 147.32 107.95 180)
-		(fields_autoplaced yes)
-		(effects
-			(font
-				(size 1.27 1.27)
-			)
-			(justify right)
-		)
-	)
-	(hierarchical_label "SCLK"
-		(shape input)
-		(at 147.32 105.41 180)
-		(fields_autoplaced yes)
-		(effects
-			(font
-				(size 1.27 1.27)
-			)
-			(justify right)
-		)
-	)
-	(hierarchical_label "3.0V"
-		(shape passive)
-		(at 109.22 83.82 0)
-		(fields_autoplaced yes)
-		(effects
-			(font
-				(size 1.27 1.27)
-			)
-			(justify left)
-		)
-	)
 	(symbol
 		(lib_id "Device:C_Small")
@@
 	)
 	(symbol
+		(lib_id "power:+1V8")
+		(at 152.4 77.47 90)
+		(unit 1)
+		(exclude_from_sim no)
+		(in_bom yes)
+		(on_board yes)
+		(dnp no)
+		(fields_autoplaced yes)
+		(property "Reference" "#PWR073"
+			(at 156.21 77.47 0)
+			(effects
+				(font
+					(size 1.27 1.27)
+				)
+				(hide yes)
+			)
+		)
+		(property "Value" "+1V8"
+			(at 148.59 77.4699 90)
+			(effects
+				(font
+					(size 1.27 1.27)
+				)
+				(justify left)
+			)
+		)
+		(property "Footprint" ""
+			(at 152.4 77.47 0)
+			(effects
+				(font
+					(size 1.27 1.27)
+				)
+				(hide yes)
+			)
+		)
+		(property "Datasheet" ""
+			(at 152.4 77.47 0)
+			(effects
+				(font
+					(size 1.27 1.27)
+				)
+				(hide yes)
+			)
+		)
+		(property "Description" "Power symbol creates a global label with name \"+1V8\""
+			(at 152.4 77.47 0)
+			(effects
+				(font
+					(size 1.27 1.27)
+				)
+				(hide yes)
+			)
+		)
+		(pin "1"
+		)
+		(instances
+			(project ""
+				(path "/110ea5a2-03d6-426d-b79f-fcb4ea6cee9d/67feebfd-a6ea-41ab-b461-383184077ed3"
+					(reference "#PWR073")
+					(unit 1)
+				)
+			)
+		)
+	)
+	(symbol
 		(lib_id "Library:FAN5331SX")
 		(at 82.55 86.36 0)
@@
 					(unit 1)
 				)
+			)
+		)
+	)
+	(symbol
+		(lib_id "power:+3V0")
+		(at 109.22 83.82 0)
+		(unit 1)
+		(exclude_from_sim no)
+		(in_bom yes)
+		(on_board yes)
+		(dnp no)
+		(fields_autoplaced yes)
+		(property "Reference" "#PWR072"
+			(at 109.22 87.63 0)
+			(effects
+				(font
+					(size 1.27 1.27)
+				)
+				(hide yes)
+			)
+		)
+		(property "Value" "+3V0"
+			(at 109.22 78.74 0)
+			(effects
+				(font
+					(size 1.27 1.27)
+				)
+			)
+		)
+		(property "Footprint" ""
+			(at 109.22 83.82 0)
+			(effects
+				(font
+					(size 1.27 1.27)
+				)
+				(hide yes)
+			)
+		)
+		(property "Datasheet" ""
+			(at 109.22 83.82 0)
+			(effects
+				(font
+					(size 1.27 1.27)
+				)
+				(hide yes)
+			)
+		)
+		(property "Description" "Power symbol creates a global label with name \"+3V0\""
+			(at 109.22 83.82 0)
+			(effects
+				(font
+					(size 1.27 1.27)
+				)
+				(hide yes)
+			)
+		)
+		(pin "1"
+		)
+		(instances
+			(project ""
+				(path "/110ea5a2-03d6-426d-b79f-fcb4ea6cee9d/67feebfd-a6ea-41ab-b461-383184077ed3"
+					(reference "#PWR072")
+					(unit 1)
+				)
